Commit message: H2 팔 제어·IK 를 xr_teleoperate 817fb00 H2_ArmController / H2_ArmIK 와 같게
- robots/h2: URDF·메시를 공식 assets/h2 로 교체 (0c1b4a2 팔 관절 한계 축소, 관절 원점·축은 이전과 같음),
  IK 캐시 이름 변경 (예전 캐시 미사용)
- robot.yaml ik.cost: 공식 H2 비용 50 / 0.8 / 0.01 / 0.1 (G1 은 기존 값 그대로)
- joints: 초기화 슬롯 0–34, weak 5/11 + 어깨·팔꿈치, 허리 12 roll / 13 pitch / 14 yaw,
  waist_hold_initial (허리는 시작 각도 유지, 명령 안 함)
- gains: 허리·머리 300/5, arm_velocity_limit 30 rad/s
- 클래스 이름 ArmController / ArmIK (G1_29_* 는 별칭), 공식과 다른 점은 EnableArmSDK 호출뿐 (실기 필요)
- arm_server /freeze: 허리 슬롯 하드코딩 대신 sync_targets_to_current
- robot_server: 허리 고정이면 리셋 생략, 잡기 시작 전 모드 전환 대기 자세 이동이 끝날 때까지 대기
  (허리 리셋 2 초가 없어지며 드러난 409 경합)
- utils/check_h2_official.py: 공식 클래스와 LowCmd 35 슬롯·IK 결과 비교 (전부 동일)
- G1: check_g1_equiv 전부 동일

Co-Authored-By: Claude Opus 5.5 <noreply@anthropic.com>
Claude-Session: https://claude.ai/code/session_01D2YCPi7df1ZjyDrhteYrPH

File: robots/h2/H2.urdf (robot description, URDF)
Before this commit: robot H2, 37 links, 36 joints
Links:
- removed link camera
- removed link imu_in_pelvis
- removed link imu_in_torso
- removed link left_hand_link
- removed link right_hand_link
- link left_wrist_yaw_link: mass 0.19722487 -> 0.61608207
- link right_wrist_yaw_link: mass 0.19722487 -> 0.6160821
Joints:
- removed joint camera
- removed joint imu_in_pelvis_joint
- removed joint imu_in_torso_joint
- removed joint left_hand_joint
- removed joint right_hand_joint
- joint left_elbow_joint: limit lower=-0.986 upper=3.071 effort=60 velocity=18.7 -> lower=-0.986 upper=1.60 effort=60 velocity=18.7
- joint left_shoulder_pitch_joint: limit lower=-2.618 upper=1.833 effort=130 velocity=21.9 -> lower=-2.618 upper=1.20 effort=130 velocity=21.9
- joint left_shoulder_roll_joint: limit lower=-0.517 upper=2.494 effort=60 velocity=18.7 -> lower=-0.517 upper=1.80 effort=60 velocity=18.7
- joint left_shoulder_yaw_joint: limit lower=-2.618 upper=2.618 effort=60 velocity=18.7 -> lower=-1.57 upper=1.57 effort=60 velocity=18.7
- joint left_wrist_roll_joint: limit lower=-2.618 upper=2.618 effort=60 velocity=18.7 -> lower=-1.65 upper=1.65 effort=60 velocity=18.7
- joint right_elbow_joint: limit lower=-0.986 upper=3.071 effort=60 velocity=18.7 -> lower=-0.986 upper=1.60 effort=60 velocity=18.7
- joint right_shoulder_pitch_joint: limit lower=-2.618 upper=1.833 effort=130 velocity=21.9 -> lower=-2.618 upper=1.20 effort=130 velocity=21.9
- joint right_shoulder_roll_joint: limit lower=-2.494 upper=0.517 effort=60 velocity=18.7 -> lower=-1.80 upper=0.517 effort=60 velocity=18.7
- joint right_shoulder_yaw_joint: limit lower=-2.618 upper=2.618 effort=60 velocity=18.7 -> lower=-1.57 upper=1.57 effort=60 velocity=18.7
- joint right_wrist_roll_joint: limit lower=-2.618 upper=2.618 effort=60 velocity=18.7 -> lower=-1.65 upper=1.65 effort=60 velocity=18.7
